Commit message: Fixed urdf pkg name

File: rm_pioneer_description/urdf/gimbal.urdf.xacro (robot description, xacro)
@@ -24,5 +24,5 @@
       <origin xyz="0 0 0" rpy="0 0 0" />
       <geometry>
-        <mesh filename="package://pioneer_description/meshes/yaw_link.stl" />
+        <mesh filename="package://rm_pioneer_description/meshes/yaw_link.stl" />
       </geometry>
       <material name="black"/>
@@ -31,5 +31,5 @@
       <origin xyz="0 0 0" rpy="0 0 0" />
       <geometry>
-        <mesh filename="package://pioneer_description/meshes/yaw_link.stl" />
+        <mesh filename="package://rm_pioneer_description/meshes/yaw_link.stl" />
       </geometry>
     </collision>
@@ -50,5 +50,5 @@
       <origin xyz="0 0 0" rpy="0 0 0" />
       <geometry>
-        <mesh filename="package://pioneer_description/meshes/pitch_link.stl" />
+        <mesh filename="package://rm_pioneer_description/meshes/pitch_link.stl" />
       </geometry>
       <material name="gray"/>
@@ -57,5 +57,5 @@
       <origin xyz="0 0 0" rpy="0 0 0" />
       <geometry>
-        <mesh filename="package://pioneer_description/meshes/pitch_link.stl" />
+        <mesh filename="package://rm_pioneer_description/meshes/pitch_link.stl" />
       </geometry>
     </collision>
