Commit message: Update guard description

File: rm_pioneer_description/urdf/guard.urdf.xacro (robot description, xacro)
@@ -5,15 +5,15 @@
     <link name="yaw_link">
         <inertial>
-            <origin xyz="-0.026886 -0.023348 0.1049" rpy="0 0 0" />
-            <mass value="1.1684" />
-            <inertia ixx="0.0016395" ixy="7.3117E-07" ixz="0.00029349" iyy="0.0022548" iyz="-4.057E-06" izz="0.0011708" />
+            <origin xyz="6.5483E-08 -0.050209 -0.056865" rpy="0 0 0" />
+            <mass value="0.54474" />
+            <inertia ixx="0.00022219" ixy="-5.1209E-08" ixz="3.7372E-08" iyy="0.00026122" iyz="1.1456E-05" izz="0.0002457" />
         </inertial>
         <visual>
             <origin xyz="0 0 0" rpy="0 0 0" />
             <geometry>
-                <mesh filename="package://rm_pioneer_description/meshes/hero/yaw_link.stl" />
+                <mesh filename="package://rm_pioneer_description/meshes/guard/yaw_link.stl" />
             </geometry>
-            <material name="black">
-                <color rgba="0.3 0.3 0.3 1"/>
+            <material name="">
+                <color rgba="0.89804 0.91765 0.92941 1" />
             </material>
         </visual>
@@ -21,5 +21,5 @@
             <origin xyz="0 0 0" rpy="0 0 0" />
             <geometry>
-                <mesh filename="package://rm_pioneer_description/meshes/hero/yaw_link.stl" />
+                <mesh filename="package://rm_pioneer_description/meshes/guard/yaw_link.stl" />
             </geometry>
         </collision>
@@ -33,15 +33,15 @@
     <link name="pitch_link">
         <inertial>
-            <origin xyz="0.091213 0.0022754 0.01373" rpy="0 0 0" />
-            <mass value="1.237" />
-            <inertia ixx="0.00067034" ixy="8.0868E-07" ixz="-1.3744E-05" iyy="0.0016262" iyz="-2.3281E-06" izz="0.0019309" />
+            <origin xyz="0.023038 -0.00034952 -0.022985" rpy="0 0 0" />
+            <mass value="1.209" />
+            <inertia ixx="0.00096057" ixy="-7.7082E-06" ixz="-1.5997E-06" iyy="0.0013203" iyz="4.1017E-07" izz="0.0020944" />
         </inertial>
         <visual>
             <origin xyz="0 0 0" rpy="0 0 0" />
             <geometry>
-                <mesh filename="package://rm_pioneer_description/meshes/hero/pitch_link.stl" />
+                <mesh filename="package://rm_pioneer_description/meshes/guard/pitch_link.stl" />
             </geometry>
-            <material name="gray">
-                <color rgba="0.75294 0.75294 0.75294 1" />
+            <material name="">
+                <color rgba="0.89804 0.91765 0.92941 1" />
             </material>
         </visual>
@@ -49,10 +49,10 @@
             <origin xyz="0 0 0" rpy="0 0 0" />
             <geometry>
-                <mesh filename="package://rm_pioneer_description/meshes/hero/pitch_link.stl" />
+                <mesh filename="package://rm_pioneer_description/meshes/guard/pitch_link.stl" />
             </geometry>
         </collision>
     </link>
     <joint name="pitch_joint" type="revolute">
-        <origin xyz="-0.041042 0 0.17276" rpy="0 0 0" />
+        <origin xyz="0 0.003 -0.074" rpy="0 0 0" />
         <parent link="yaw_link" />
         <child link="pitch_link" />
@@ -62,5 +62,5 @@
     <link name="shooter_link" />
     <joint name="shooter_joint" type="fixed">
-        <origin xyz="-0.041042 0 0.17276" rpy="0 0 0" />
+        <origin xyz="0 0.003 -0.074" rpy="0 0 0" />
         <parent link="base_link" />
         <child link="shooter_link" />
@@ -68,15 +68,15 @@
     <link name="camera_base_link">
         <inertial>
-            <origin xyz="0.014834 -3.0881E-18 0" rpy="0 0 0" />
-            <mass value="0.052061" />
-            <inertia ixx="6.6064E-06" ixy="2.1459E-21" ixz="-1.7784E-21" iyy="2.3578E-05" iyz="-2.5012E-22" izz="2.3576E-05" />
+            <origin xyz="-5.2307E-05 -1.5998E-05 0.00049253" rpy="0 0 0" />
+            <mass value="0.15794" />
+            <inertia ixx="7.7178E-05" ixy="-7.743E-08" ixz="-1.6158E-07" iyy="0.00010028" iyz="-2.0158E-08" izz="0.00010682" />
         </inertial>
         <visual>
             <origin xyz="0 0 0" rpy="0 0 0" />
             <geometry>
-                <mesh filename="package://rm_pioneer_description/meshes/hero/camera_base_link.stl" />
+                <mesh filename="package://rm_pioneer_description/meshes/guard/camera_base_link.stl" />
             </geometry>
-            <material name="cyan">
-                <color rgba="0.3 0.7 0.8 1"/>
+            <material name="">
+                <color rgba="1 1 1 1" />
             </material>
         </visual>
@@ -84,10 +84,10 @@
             <origin xyz="0 0 0" rpy="0 0 0" />
             <geometry>
-                <mesh filename="package://rm_pioneer_description/meshes/hero/camera_base_link.stl" />
+                <mesh filename="package://rm_pioneer_description/meshes/guard/camera_base_link.stl" />
             </geometry>
         </collision>
     </link>
-    <joint name="camera_base_joint" type="fixed">
-        <origin xyz="0.15839 0 -0.05" rpy="0 0 0" />
+    <joint name="camera_joint" type="fixed">
+        <origin xyz="0.132 0 -0.048" rpy="0 0 0" />
         <parent link="pitch_link" />
         <child link="camera_base_link" />

File: rm_pioneer_description/urdf/standard.urdf.xacro (robot description, xacro)
@@ -9,10 +9,4 @@
   </material>
   <link name="base_link" />
-  <link name="shooter_link" />
-  <joint name="shooter_joint" type="fixed">
-    <origin xyz="0 0 0.137" rpy="0 0 0" />
-    <parent link="base_link" />
-    <child link="shooter_link" />
-  </joint>
   <link name="yaw_link">
     <inertial>
@@ -68,4 +62,10 @@
     <limit lower="-0.6" upper="0.5" effort="1.2" velocity="31"/>
   </joint>
+  <link name="shooter_link" />
+  <joint name="shooter_joint" type="fixed">
+    <origin xyz="0 0 0.137" rpy="0 0 0" />
+    <parent link="base_link" />
+    <child link="shooter_link" />
+  </joint>
   <link name="camera_base_link" />
   <joint name="camera_base_joint" type="fixed">
